Commit message: feat(edu1): widen joint4 to ±115°, and replace the proof that widening killed
The Edu:1's wrist pitch was ±90° (1.5708 rad). The hardware reaches ±115° —
the owner's statement, not a measurement this repo can make — so ±115° is a
CEILING, and 2.0071 rounds INWARD of it by 2.864e-5 rad ≈ 0.019 servo ticks,
keeping the shipped URDF's four-decimal convention.

WHY: joint2/3/4 are parallel, so for a strict-vertical claw q4 is DETERMINED
(q4 = q2 − q3 + BETA0 − π) and always NEGATIVE — only the lower limit ever
clips it. Measured through the real solver over r ∈ [0.05, 0.40] × z ∈
[0.00, 0.40] at 5 mm (5751 cells): 902 → 2068 cells solved, strict-vertical
ceiling 0.100 m → 0.195 m, and the window admits 29.2 % → 67.0 % of the
2R-feasible set (required q4 spans −171.21°…−62.86°).

THE PROOF THIS BREAKS. edu1_ik.solve carried an in-code proof that the
elbow-down branch is unreachable, and it consumed `q4 ≥ −π/2`. That premise is
now false and the proof genuinely fails: elbow-down IS in limits over a real
region (4118 cells of a 900×900 (g, ψ) enumeration at z ≥ 0; 17 of the 4000
targets the shipped test samples, which is why that test failed and had to
change). The branch is still never SELECTED, for a reason that never depended
on the bound: writing φ for the 2R triangle's shoulder angle,

    q4_up − q4_down = 2(|g| − |φ|) = 2 × the triangle's WRIST interior angle > 0

and q2_down ≥ q2_up, q3_down ≥ q3_up. So elbow-down being in limits IMPLIES
elbow-up is too, and elbow-up is tried first. Holds for any window ≥ ±0.20295
rad and uses no property of z. Confirmed three ways: the algebra against the
solver's own expressions (max err 1.3e-15 over 200k samples), the exhaustive
enumeration (4118/4118 also elbow-up, 0 elbow-down-only), and a direct 260×260
solve() sweep (23359/23359 elbow-up, 0 elbow-down).

So the posture the arm adopts is UNCHANGED — which is what every clearance
figure and path_guard's "no reconfiguration flip" rest on. The test now asserts
that property directly instead of the old proxy ("never in limits"), plus the
dominance lemma, and carries a guard that fails if the sample stops covering
the region where the two differ.

SAFETY, re-measured over the NEW pose space (shipped oracle, seed 4242):
floor-clearance model sound 400/400 (reproducing the shipped ±90° figure
exactly: median 0.00, mean 12.80, p95 50.97, max 71.08 mm), and at ±115°
400/400, 2000/2000, and 20000/20000 with q4 drawn ONLY from the newly opened
bands (median 0.00, mean 11.90, p95 52.72, max 74.87 mm). Self-clearance vs a
decimated mesh oracle: sound 40/40. Soundness is also structural — each box is
an AABB of its link's mesh in that link's OWN frame, so mesh ⊆ box holds for
every pose. HOME (0, 0.64, 1.48, 0.90, 0) stays in the window and its binding
joint is still joint2 at 0.640 rad, so its objective is unchanged.

⚠ RE-PROVISIONING IS MANDATORY. The driver's boot probe verifies the servo
EEPROM Min/Max_Position_Limit window as a provisioning fingerprint. joint4's
window moves 1024…3072 → 740…3356 ticks, so every physical Edu:1 must be re-run
through `tools/edu6_provision.py --arm edu1` or it will refuse to boot, in
German, with no hint why.

The pair is declared in FOUR cross-pinned places and all four move here: the
shipped URDF, edu1_ik.py, edu6_arm_node.py and edu6_provision.py. Reverting any
one alone is caught by an existing test (verified, one site at a time).

Also fixed, found while re-deriving:
* test_edu1_ik.py had a HARD-CODED `-1.5708 <= q4 <= 1.5708` sample filter, so
  it would have kept testing only the old window while staying green. It now
  reads the constant.
* robot_profiles said the swing grid gives "32/72" six lines above saying
  "36/72". Measured 36/72, at both windows.
* reach_inner_m 0.09 → 0.07. The ring rule is now the INTERSECTION of the grasp
  plane and the hover the catalog asks for, not the grasp plane alone: the old
  rim r=0.35 was solvable only to z ≈ 0.033, i.e. 18 mm of hover against a
  60 mm request, bisected on every rim grasp and silently (the clamp only warns
  below 15 mm). At ±115° r=0.35 reaches z ≈ 0.093 and gets the full 60 mm. The
  outer deliberately does NOT go to the new grasp-plane edge 0.37, which would
  hand the rim straight back its silent clamp.
* the edu1 URDF header's "12 non-ASCII bytes" was already wrong at HEAD (21).

OMX and edu6 are bit-identical: a sha256 over 10 800 solve() calls per arm
(60×60 grid × 3 rolls), FK, capabilities_json, profile geometry and
resolve_geometry's None-ness matches HEAD exactly, and dof_golden.json is
untouched. Suites: server 1694 passed / 4 skipped (baseline 1693, +1 new test),
GUI 1397 OK (skipped=9), pi_agent 587 OK.

Co-Authored-By: Claude Opus 5 (1M context) <noreply@anthropic.com>
Claude-Session: https://claude.ai/code/session_01Jt46Zb9BBeDexFBLs7Tpks

File: physical_ai_tools/physical_ai_manager/public/edu1-urdf/edu1.urdf (robot description, URDF)
Before this commit: robot edu1_studio, 9 links, 8 joints
Joints:
- joint joint4: limit lower=-1.5708 upper=1.5708 effort=1.91 velocity=4.72 -> lower=-2.0071 upper=2.0071 effort=1.91 velocity=4.72
